File: DAQ.kicad_sch (KiCad schematic)
At the start: 141 parts, among them J1 ICD15S13E4GX00LF, J2 ICD15S13E4GX00LF, J3 ICD15S13E4GX00LF, P1 0022272021, U1 ADS124S08IRHBT, U2 ADS124S08IRHBT, U3 LT6654BMPS6-5-TRMPBF, U4 LM1086IS-5.0_NOPB, U5 TPS73801DCQR, U6 TPSM63603RDHR, U7 TPSM63603RDHR, U8 TPSM63603RDHR

Commit message: Clean up schematic
Parts:
- C1, C10, C11, C12, C13, C14, C15, C16, C17, C18, C19, C2, C20, C21, C22, C23, C24, C25, C26, C27, C28, C29, C3, C30, C31, C32, C33, C34, C35, C36, C37, C38, C39, C4, C41, C43, C45, C46, C47, C48, C49, C5, C50, C51, C52, C53, C54, C55, C56, C57, C58, C59, C6, C60, C61, C62, C63, C64, C65, C66, C67, C68, C69, C7, C70, C71, C72, C73, C74, C8, C9, D1, D2, D3, D4, D5, D6, D7, D8, H1, H2, H3, H4, J1, J2, J3, P1, R1, R10, R11, R12, R13, R14, R15, R16, R17, R18, R19, R2, R20, R21, R22, R23, R24, R25, R26, R29, R3, R30, R31, R32, R33, R34, R35, R36, R37, R38, R39, R4, R40, R5, R6, R7, R8, R9, U2, U3, U4, U5, U6, U7, U8: now fitted

Commit message: Added differential amplifiers
Parts:
- removed C21, C22, C23: 16nF, GRM3195C2A163JA01D:CAPC3216X95N, symbol Device:C
- removed R14, R15, R16: 10k, footprints10kR:RC0603N_YAG-M, symbol Device:R
- added U10, U11, U9: INA105KU_2K5, INA105KU_2K5:SOIC127P599X175-8N, symbol INA105KU_2K5:INA105KU_2K5
- C15: value 16nF -> 1uF; footprint GRM3195C2A163JA01D:CAPC3216X95N -> 0603YC105JAT2A:CAPC1608X94N
- C7: value 3.3nF -> 16nF; footprint footprintsCL10:CAP_CL10_SAM -> GRM3195C2A163JA01D:CAPC3216X95N
- C8, C9: value 3.3nF -> 1uF; footprint footprintsCL10:CAP_CL10_SAM -> 0603YC105JAT2A:CAPC1608X94N
- R11, R12, R13: value 10k -> ~1k (LOOK INTO THIS LOW PASS FILTER)
Connections:
- net +5Vs: no longer D5.6, D6.4
- net 10Vs: no longer D7.1 (K_1)
- net 24V: now also C15.1, C8.1, C9.1, U10.7 (V+), U11.7 (V+), U9.7 (V+)
- net GND: now also C7.2, C8.2, C9.2, U10.1 (REF), U10.4 (V-), U11.1 (REF), U11.4 (V-), U9.1 (REF), U9.4 (V-)
- net LS1_SIG+: no longer J1.3, R11.1
- net LS1_SIG-: no longer J1.2, R12.1
- net LS2_SIG+: no longer J1.10, R13.1
- net LS2_SIG-: no longer J1.15
- net LS3_SIG+: no longer J2.11
- net LS3_SIG-: no longer J2.12
- net LC1_SIG: now reaches C7.1, R11.2, U1.6 (AIN1)
- net LC1_SIG: no longer C14.1
- net LC2_SIG: now reaches R12.2, U1.7 (AIN0)
- net LC2_SIG: now also C14.1; no longer C7.2
- net LC3_SIG: now reaches R13.2, U1.19 (GPIO3_AIN11)
- net LC3_SIG: now also C16.1; no longer C15.1, C8.1
- net at U1.20 (GPIO2_AIN10): no longer C8.2
- net at U1.22 (GPIO0_AIN8): no longer C9.2
- new net: R12.1, U10.5 (SENSE), U10.6 (OUT)
- new net: R13.1, U11.5 (SENSE), U11.6 (OUT)
- new net: R11.1, U9.5 (SENSE), U9.6 (OUT)
- new net LC1_SIG+: J1.3, U9.3 (+IN)
- new net LC1_SIG-: J1.2, U9.2 (-IN)
- new net LC2_SIG+: J1.10, U10.3 (+IN)
- new net LC2_SIG-: J1.15, U10.2 (-IN)
- new net LC3_SIG+: J2.11, U11.3 (+IN)
- new net LC3_SIG-: J2.12, U11.2 (-IN)
- new net LS1_EXCT+: D7.1 (K_1)
- new net LS2_EXCT+: D6.4
- new net LS3_EXCT+: D5.6
- now unconnected: U1.21 (GPIO1_AIN9)
- no-connect marks 36 -> 39
Other:
- moved on the sheet: C46, C47, C48, C49, C50, C51, C52, C53, C54, C55, C56, C57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
